File: picothermal-hardware/picothermal-hardware.kicad_pcb (KiCad board)
At the start: 4 copper layers, 50 x 30 mm, 118 parts, among them J1 TC2030-CTX, J2 USB-C Plug, SW1 SW_Push, SW2 SW_Push, U1 W25Q16JV, U2 AP7330-W5-7, U3 AP7330-W5-7, U4 RP2040, U5 TLV62569A, U6 TLV62569A, U7 Flir LEPTON, Y1 ECS-2520MV-250-CL, Y2 12MHz

Commit message: Final review passed and added fabrication outputs
Parts:
- added kibuzzard-63AA0E75: G***, kibuzzard-63AA0E75, F.Cu at (109.9, 108.0)
- added kibuzzard-63AA0EB3: G***, kibuzzard-63AA0EB3, F.Cu at (81.0, 108.0)
- added kibuzzard-63AA0F05: G***, kibuzzard-63AA0F05, F.Cu at (92.4, 109.8)
- moved R3 0.65 mm to (85.7, 112.0), turned to 180 degrees
- moved C21 0.18 mm to (114.3, 105.1)
- moved C8 0.15 mm to (105.9, 101.2)
- moved C23 0.12 mm to (105.9, 100.3)
- moved R21 0.12 mm to (113.4, 105.1)
- moved C9 0.10 mm to (118.0, 97.8)
- moved C14 0.10 mm to (105.9, 99.5)
- moved R18 0.08 mm to (112.6, 105.1)
- moved R6 0.05 mm to (105.9, 98.7)
Routing:
- net GND: track 15.0 -> 20.2 mm, vias 91 -> 100
- net +3V0: track 51.3 -> 55.8 mm
- net +2V8: track 39.2 -> 42.6 mm
- net +1V1: track 26.7 -> 28.2 mm
- net /GPIO_SW: track 40.7 -> 39.3 mm
- net +5V: vias 21 -> 23
Other:
- board text removed: "BOOT"
- board text removed: "Picothermal"
- board text removed: "SWITCH"
